Commit message: Update panda model

File: urdfs/panda.urdf (robot description, URDF)
Before this commit: robot panda, 14 links, 13 joints
Links:
- added link camera_base; visual box size=0.026 0.103 0.039
- added link camera_body; visual box size=0.0994 0.0996 0.023
- added link camera_visor; visual box size=0.026 0.101 0.037
Joints:
- added joint camera_base_to_body: type fixed, parent camera_base, child camera_body, origin xyz=-0.0757 0. 0.008 rpy=0. 0. 0.
- added joint camera_base_to_visor: type fixed, parent camera_base, child camera_visor, origin xyz=0. 0. 0. rpy=0. 0. 0.
- added joint fake_base: type fixed, parent panda_link6, child camera_base, origin xyz=0.156 -0.052 -0.005 rpy=-1.586 0.010 -1.585

Commit message: Prepare simu only

File: urdfs/panda.urdf (robot description, URDF)
Before this commit: robot panda_kinect, 17 links, 16 joints
Links:
- removed link end_effector
Joints:
- removed joint end_effector
- joint fake_base: origin xyz=0.156 -0.052 -0.005 rpy=-1.586 0.010 -1.585 -> xyz=0.156 -0.041 0.00 rpy=-1.586 0.010 -1.585

Commit message: Fix dependencies

File: urdfs/panda.urdf (robot description, URDF)
Before this commit: robot panda_kinect, 16 links, 15 joints
Links:
- link panda_hand: geometry collision mesh filename=package://authoring/meshes/collision/hand.stl; visual mesh filename=package://authoring/meshes/visual/hand.dae
- link panda_leftfinger: geometry collision mesh filename=package://authoring/meshes/collision/finger.stl; visual mesh filename=package://authoring/meshes/visual/finger.dae
- link panda_link0: geometry collision mesh filename=package://authoring/meshes/collision/link0.stl; visual mesh filename=package://authoring/meshes/visual/link0.dae
- link panda_link1: geometry collision mesh filename=package://authoring/meshes/collision/link1.stl; visual mesh filename=package://authoring/meshes/visual/link1.dae
- link panda_link2: geometry collision mesh filename=package://authoring/meshes/collision/link2.stl; visual mesh filename=package://authoring/meshes/visual/link2.dae
- link panda_link3: geometry collision mesh filename=package://authoring/meshes/collision/link3.stl; visual mesh filename=package://authoring/meshes/visual/link3.dae
- link panda_link4: geometry collision mesh filename=package://authoring/meshes/collision/link4.stl; visual mesh filename=package://authoring/meshes/visual/link4.dae
- link panda_link5: geometry collision mesh filename=package://authoring/meshes/collision/link5.stl; visual mesh filename=package://authoring/meshes/visual/link5.dae
- link panda_link6: geometry collision mesh filename=package://authoring/meshes/collision/link6.stl; visual mesh filename=package://authoring/meshes/visual/link6.dae
- link panda_link7: geometry collision mesh filename=package://authoring/meshes/collision/link7.stl; visual mesh filename=package://authoring/meshes/visual/link7.dae
- link panda_rightfinger: geometry collision mesh filename=package://authoring/meshes/collision/finger.stl; visual mesh filename=package://authoring/meshes/visual/finger.dae

Commit message: Update camera position

File: urdfs/panda.urdf (robot description, URDF)
Before this commit: robot panda_kinect, 16 links, 15 joints
Links:
- link camera_base: geometry 
- link camera_body: geometry visual mesh filename=package://authoring/meshes/visual/kinect-model.stl
- link camera_visor: geometry 
Joints:
- joint fake_base: origin xyz=0.156 -0.041 0.00 rpy=-1.586 0.010 -1.585 -> xyz=0.025 -0.065 0.01 rpy=3.14 -1.57 -0.785; parent panda_link6 -> panda_link8

Commit message: Camera calibration

File: urdfs/panda.urdf (robot description, URDF)
Before this commit: robot panda_kinect, 16 links, 15 joints
Joints:
- joint fake_base: origin xyz=0.025 -0.065 0.01 rpy=3.14 -1.57 -0.785 -> xyz=0.029 -0.056 0.01 rpy=3.14 -1.57 -0.785
