Commit message: Forgotten end_effect -> panda_gripper

File: urdfs/panda_arm_hand.urdf (robot description, URDF)
Before this commit: robot panda, 14 links, 13 joints
Links:
- removed link end_effector
- added link panda_gripper
Joints:
- removed joint end_effector
- added joint panda_gripper: type fixed, parent panda_link8, child panda_gripper, origin xyz=-0.000 -0.000 0.103 rpy=-0.000 0.000 -0.785, axis 0 0 0
